Commit message: [ADD] new items inside washing machine

File: worlds/rcjo2026_arena.world.xacro (robot description, xacro)
@@ -98,6 +98,6 @@
       <!-- OPEN: panel alongside inner face of wall_front_right (y≈-3.0),
            reaching 0.9 m into the arena from the front wall (x=-5.0→-4.1) -->
-      <!-- <pose>-4.55 -3.0 1.0 0.0 0.0 0.0</pose> -->
-      <pose>-4.55 2.0 1.0 0.0 0.0 0.0</pose>
+      <!-- <pose>-4.55 2.0 1.0 0.0 0.0 0.0</pose> -->
+      <pose>-5.0 1.5 1.0 0 0 1.5708</pose>
       <link name="panel">
         <collision name="col">
@@ -172,4 +172,34 @@
       <pose relative_to=''>2.3 -3.2 0.15 0.0 0.0 0.0</pose>
     </include>
+    <!-- Laundry cloth in drum — rigid box proxy for fabric (Gazebo cloth not supported).
+         Washing machine is at (1.375, -3.5, 0.0) yaw=π/2, so the drum door faces world +Y.
+         This places the proxy inside the drum: same X as washer, 0.2 m toward room along
+         the drum axis (Y=-3.3), at the drum interior height (Z=0.55).
+         Name MUST be "laundry_in_drum" — stubs_node publishes TF "laundry_in_drum_0". -->
+    <model name="laundry_in_drum">
+      <static>false</static>
+      <pose>1.375 -3.5 0.55 0 0 0</pose>
+      <link name="link">
+        <inertial>
+          <mass>0.3</mass>
+          <inertia>
+            <ixx>0.001</ixx><ixy>0</ixy><ixz>0</ixz>
+            <iyy>0.001</iyy><iyz>0</iyz>
+            <izz>0.001</izz>
+          </inertia>
+        </inertial>
+        <collision name="collision">
+          <geometry><box><size>0.15 0.10 0.05</size></box></geometry>
+        </collision>
+        <visual name="visual">
+          <geometry><box><size>0.15 0.10 0.05</size></box></geometry>
+          <material>
+            <ambient>0.2 0.4 0.8 1</ambient>
+            <diffuse>0.2 0.4 0.8 1</diffuse>
+            <specular>0.05 0.05 0.05 1</specular>
+          </material>
+        </visual>
+      </link>
+    </model>
     <!-- Living Room / Laundry Area -->
     <!-- Study Room -->
