Commit message: [ADD&UPDATE]Add folded shirt models and update laundry world

File: worlds/doing_laundry.world.xacro (robot description, xacro)
@@ -1,10 +1,4 @@
 <?xml version="1.0" ?>
 <sdf version="1.8" xmlns:xacro="http://www.ros.org/wiki/xacro">
-  <!-- Doing Laundry world (template)
-       - Entrance door is represented by a removable "blocker" model:
-         model name: entrance_door_blocker
-       - After Gazebo starts, remove that model via:
-         /world/<world_name>/remove  (gz service)
-  -->
   <world name='doing_laundry_arena'>
     <plugin filename="gz-sim-physics-system"        name="gz::sim::systems::Physics"/>
@@ -12,7 +6,5 @@
     <plugin filename="gz-sim-scene-broadcaster-system" name="gz::sim::systems::SceneBroadcaster"/>
     <plugin filename="gz-sim-sensors-system"        name="gz::sim::systems::Sensors"/>
-    <scene>
-      <grid>false</grid>
-    </scene>
+    <scene><grid>false</grid></scene>
     <physics name="1ms" type="ignored">
       <max_step_size>0.001</max_step_size>
@@ -21,129 +13,101 @@
     <light type="directional" name="sun">
       <cast_shadows>true</cast_shadows>
-      <pose relative_to=''>0 0 10 0 0 0</pose>
+      <pose>0 0 10 0 0 0</pose>
       <diffuse>0.8 0.8 0.8 1</diffuse>
       <specular>0.2 0.2 0.2 1</specular>
-      <attenuation>
-        <range>1000</range>
-        <constant>0.9</constant>
-        <linear>0.01</linear>
-        <quadratic>0.001</quadratic>
-      </attenuation>
       <direction>-0.5 0.1 -0.9</direction>
     </light>
     <gravity>0 0 -9.8</gravity>
     <!-- Floor -->
-    <include>
-      <name>floor_plane_fl</name>
-      <static>1</static>
-      <uri>model://wrc_ground_plane</uri>
-      <pose relative_to=''>5 5 0 0 0 0</pose>
-    </include>
-    <include>
-      <name>floor_plane_fr</name>
-      <static>1</static>
-      <uri>model://wrc_ground_plane</uri>
-      <pose relative_to=''>5 -5 0 0 0 0</pose>
-    </include>
-    <include>
-      <name>floor_plane_bl</name>
-      <static>1</static>
-      <uri>model://wrc_ground_plane</uri>
-      <pose relative_to=''>-5 5 0 0 0 0</pose>
-    </include>
-    <include>
-      <name>floor_plane_br</name>
-      <static>1</static>
-      <uri>model://wrc_ground_plane</uri>
-      <pose relative_to=''>-5 -5 0 0 0 0</pose>
-    </include>
-    <!-- Optional frame -->
+    <include><name>floor_plane_fl</name><static>1</static><uri>model://wrc_ground_plane</uri><pose> 5  5 0 0 0 0</pose></include>
+    <include><name>floor_plane_fr</name><static>1</static><uri>model://wrc_ground_plane</uri><pose> 5 -5 0 0 0 0</pose></include>
+    <include><name>floor_plane_bl</name><static>1</static><uri>model://wrc_ground_plane</uri><pose>-5  5 0 0 0 0</pose></include>
+    <include><name>floor_plane_br</name><static>1</static><uri>model://wrc_ground_plane</uri><pose>-5 -5 0 0 0 0</pose></include>
     <include>
       <name>rcjo2025_frame</name>
       <static>1</static>
       <uri>model://rcjo2025_frame</uri>
-      <pose relative_to=''>0 0 0 0 0 0</pose>
+      <pose>0 0 0 0 0 0</pose>
     </include>
-    <!-- ============================================================= -->
-    <!-- Entrance "door" as a blocker (remove after start)              -->
-    <!-- ============================================================= -->
+    <!-- Entrance door blocker (pose matches image1) -->
     <model name="entrance_door_blocker">
       <static>true</static>
-      <!-- TODO: Adjust this pose to your actual entrance location.
-           This pose is just a placeholder.
-           z=1.0 so the 2m-high panel is centered around the doorway height.
-      -->
-      <pose>5.0 0.0 1.0 0 0 0</pose>
+      <!-- from image1 UI: x=-0.06, y=-1.98, z=1.00, r=p=yaw=0 -->
+      <pose>-0.06 -1.98 1.00 0 0 0</pose>
       <link name="link">
         <collision name="collision">
-          <geometry>
-            <!-- width>=0.90, height>=2.00 -->
-            <box><size>0.05 1.0 2.05</size></box>
-          </geometry>
+          <geometry><box><size>0.05 1.0 2.05</size></box></geometry>
         </collision>
         <visual name="visual">
-          <geometry>
-            <box><size>0.05 1.0 2.05</size></box>
-          </geometry>
-          <material>
-            <!-- slightly transparent so you can see it in GUI -->
-            <diffuse>0.2 0.2 0.2 0.6</diffuse>
-          </material>
+          <geometry><box><size>0.05 1.0 2.05</size></box></geometry>
+          <material><diffuse>0.2 0.2 0.2 0.6</diffuse></material>
         </visual>
       </link>
     </model>
-    <!-- ============================================================= -->
-    <!-- Laundry area                                                   -->
-    <!-- ============================================================= -->
-    <!-- Folding/work table -->
+    <!-- Laundry area -->
     <include>
       <name>laundry_room#folding_table</name>
       <uri>model://wrc_long_table</uri>
       <static>1</static>
-      <pose relative_to=''>2.0 -0.5 0 0 0 0</pose>
+      <pose>2.0 -0.5 0 0 0 0</pose>
     </include>
-    <!-- (optional) tall table -->
     <include>
       <name>laundry_room#tall_table</name>
       <uri>model://wrc_tall_table</uri>
       <static>1</static>
-      <pose relative_to=''>0.75 -0.5 0 0 0 0</pose>
+      <pose>0.75 -0.5 0 0 0 0</pose>
     </include>
-    <!-- Washing machine (door remains closed) -->
     <include>
       <name>washing_machine</name>
       <uri>model://washing_machine</uri>
       <static>0</static>
-      <pose relative_to=''>1.375 -3.5 0.0 0.0 0.0 1.5708</pose>
+      <pose>1.375 -3.5 0.0 0.0 0.0 1.5708</pose>
     </include>
-    <!-- Laundry basket -->
     <include>
       <name>laundry_basket</name>
       <uri>model://laundry_basket</uri>
       <static>0</static>
-      <pose relative_to=''>2.3 -3.2 0.0 0.0 0.0 0.0</pose>
+      <pose>2.3 -3.2 0.0 0.0 0.0 0.0</pose>
     </include>
-    <!-- One shirt proxy on table (add more later) -->
-    <model name="shirt_on_table_0">
-      <static>false</static>
-      <pose>2.0 -0.5 0.78 0 0 0</pose>
-      <link name="link">
-        <inertial>
-          <mass>0.2</mass>
-          <inertia>
-            <ixx>0.0005</ixx><ixy>0</ixy><ixz>0</ixz>
-            <iyy>0.0005</iyy><iyz>0</iyz>
-            <izz>0.0005</izz>
-          </inertia>
-        </inertial>
-        <collision name="collision">
-          <geometry><box><size>0.28 0.28 0.03</size></box></geometry>
-        </collision>
-        <visual name="visual">
-          <geometry><box><size>0.28 0.28 0.03</size></box></geometry>
-          <material><diffuse>0.2 0.5 0.9 1</diffuse></material>
-        </visual>
-      </link>
-    </model>
+        <!-- Folded shirts (GLB-based models) -->
+    <!-- Table (1) -->
+    <include>
+      <name>folded_shirt_table_0</name>
+      <uri>model://folded_shirt_white</uri>
+      <static>0</static>
+      <pose>2.00 -0.50 0.78 0 0 0</pose>
+    </include>
+    <!-- Washing machine (3) - TODO: tune pose to be inside drum -->
+    <include>
+      <name>folded_shirt_washer_0</name>
+      <uri>model://folded_shirt_green</uri>
+      <static>0</static>
+      <pose>1.33 -3.50 0.60 0 0 1.57</pose>
+    </include>
+    <include>
+      <name>folded_shirt_washer_1</name>
+      <uri>model://folded_shirt_white</uri>
+      <static>0</static>
+      <pose>1.40 -3.45 0.60 0 0 1.20</pose>
+    </include>
+    <include>
+      <name>folded_shirt_washer_2</name>
+      <uri>model://folded_shirt_green</uri>
+      <static>0</static>
+      <pose>1.28 -3.55 0.60 0 0 1.90</pose>
+    </include>
+    <!-- Basket (2) - TODO: tune pose to be inside basket -->
+    <include>
+      <name>folded_shirt_basket_0</name>
+      <uri>model://folded_shirt_white</uri>
+      <static>0</static>
+      <pose>2.30 -3.20 0.22 0 0 0.20</pose>
+    </include>
+    <include>
+      <name>folded_shirt_basket_1</name>
+      <uri>model://folded_shirt_green</uri>
+      <static>0</static>
+      <pose>2.35 -3.15 0.22 0 0 -0.30</pose>
+    </include>
   </world>
 </sdf>

File: worlds/rcjo2025_arena.world.xacro (robot description, xacro)
@@ -192,10 +192,10 @@
     <!-- Dining Room -->
     <!-- Bedroom -->
-    <include>
+    <!-- <include>
       <name>bedroom#sofa</name>
       <uri>model://sofa</uri>
       <static>1</static>
       <pose relative_to=''>-2.0 3.25 0.0 0.0 0.0 1.57</pose>
-    </include>
+    </include> -->
     <include>
       <name>bedroom#bed</name>
@@ -204,14 +204,21 @@
       <pose relative_to=''>-3.9 3.25 0.0 0.0 0.0 1.57</pose>
     </include>
-    <include>
+    <!-- <include>
       <name>human</name>
       <uri>model://human</uri>
       <static>1</static>
       <pose relative_to=''>-3.9 3.25 0.0 0.0 0.0 1.57</pose>
-    </include>
-    <include>
+    </include> -->
+    <include>
+      <name>bedroom#arm_chair</name>
       <uri>model://arm_chair</uri>
       <static>false</static>
-      <pose relative_to=''>-2.0 3.25 5.0 0.0 0.0 1.57</pose>
+      <pose relative_to=''>-2.0 3.25 0.0 0.0 0.0 0.0</pose>
+    </include>
+    <include>
+      <name>bedroom#apple</name>
+      <uri>model://apple</uri>
+      <static>false</static>
+      <pose relative_to='bedroom#arm_chair'>0 0 1.0 0 0 0</pose>
     </include>
     <!-- Bedroom -->

Commit message: [ADD] Implement door open/close service and update related world files

File: worlds/doing_laundry.world.xacro (robot description, xacro)
@@ -30,17 +30,33 @@
       <pose>0 0 0 0 0 0</pose>
     </include>
-    <!-- Entrance door blocker (pose matches image1) -->
-    <model name="entrance_door_blocker">
-      <static>true</static>
-      <!-- from image1 UI: x=-0.06, y=-1.98, z=1.00, r=p=yaw=0 -->
-      <pose>-0.06 -1.98 1.00 0 0 0</pose>
-      <link name="link">
+    <!-- Entrance door (open/close by pose update) -->
+    <model name="entrance_door">
+      <static>false</static>
+      <pose>0.02 -3.01 0.87 0 0 0</pose>
+      <link name="door_link">
         <collision name="collision">
-          <geometry><box><size>0.05 1.0 2.05</size></box></geometry>
+          <pose>0 1 0 0 0 0</pose>
+          <geometry>
+            <box><size>0.05 2.0 2.05</size></box>
+          </geometry>
         </collision>
         <visual name="visual">
-          <geometry><box><size>0.05 1.0 2.05</size></box></geometry>
-          <material><diffuse>0.2 0.2 0.2 0.6</diffuse></material>
+          <pose>0 1 0 0 0 0</pose>
+          <geometry>
+            <box><size>0.05 2.0 2.05</size></box>
+          </geometry>
+          <material>
+            <ambient>0.6 0.6 0.6 1</ambient>
+            <diffuse>0.6 0.6 0.6 1</diffuse>
+          </material>
         </visual>
+        <inertial>
+          <mass>10</mass>
+          <inertia>
+            <ixx>1</ixx><ixy>0</ixy><ixz>0</ixz>
+            <iyy>1</iyy><iyz>0</iyz>
+            <izz>1</izz>
+          </inertia>
+        </inertial>
       </link>
     </model>
@@ -70,43 +86,21 @@
       <pose>2.3 -3.2 0.0 0.0 0.0 0.0</pose>
     </include>
-        <!-- Folded shirts (GLB-based models) -->
-    <!-- Table (1) -->
     <include>
-      <name>folded_shirt_table_0</name>
+      <name>folded_shirt_front</name>
       <uri>model://folded_shirt_white</uri>
       <static>0</static>
-      <pose>2.00 -0.50 0.78 0 0 0</pose>
+      <pose>2.18 -0.49 0.41 1.5708  0 0</pose>
     </include>
-    <!-- Washing machine (3) - TODO: tune pose to be inside drum -->
     <include>
-      <name>folded_shirt_washer_0</name>
+      <name>folded_shirt_back_1</name>
+      <uri>model://folded_shirt_white</uri>
+      <static>0</static>
+      <pose>1.51 -0.49 0.41 1.5708  0 0</pose>
+    </include>
+    <include>
+      <name>folded_shirt_back_2</name>
       <uri>model://folded_shirt_green</uri>
       <static>0</static>
-      <pose>1.33 -3.50 0.60 0 0 1.57</pose>
-    </include>
-    <include>
-      <name>folded_shirt_washer_1</name>
-      <uri>model://folded_shirt_white</uri>
-      <static>0</static>
-      <pose>1.40 -3.45 0.60 0 0 1.20</pose>
-    </include>
-    <include>
-      <name>folded_shirt_washer_2</name>
-      <uri>model://folded_shirt_green</uri>
-      <static>0</static>
-      <pose>1.28 -3.55 0.60 0 0 1.90</pose>
-    </include>
-    <!-- Basket (2) - TODO: tune pose to be inside basket -->
-    <include>
-      <name>folded_shirt_basket_0</name>
-      <uri>model://folded_shirt_white</uri>
-      <static>0</static>
-      <pose>2.30 -3.20 0.22 0 0 0.20</pose>
-    </include>
-    <include>
-      <name>folded_shirt_basket_1</name>
-      <uri>model://folded_shirt_green</uri>
-      <static>0</static>
-      <pose>2.35 -3.15 0.22 0 0 -0.30</pose>
+      <pose>1.88 -0.49 0.41 1.5708  0 0</pose>
     </include>
   </world>
