Commit message: Fix doing_laundry world assets and remove door service

File: worlds/doing_laundry.world.xacro (robot description, xacro)
@@ -30,35 +30,4 @@
       <pose>0 0 0 0 0 0</pose>
     </include>
-    <!-- Entrance door (open/close by pose update) -->
-    <model name="entrance_door">
-      <static>false</static>
-      <pose>0.02 -3.01 0.87 0 0 0</pose>
-      <link name="door_link">
-        <collision name="collision">
-          <pose>0 1 0 0 0 0</pose>
-          <geometry>
-            <box><size>0.05 2.0 2.05</size></box>
-          </geometry>
-        </collision>
-        <visual name="visual">
-          <pose>0 1 0 0 0 0</pose>
-          <geometry>
-            <box><size>0.05 2.0 2.05</size></box>
-          </geometry>
-          <material>
-            <ambient>0.6 0.6 0.6 1</ambient>
-            <diffuse>0.6 0.6 0.6 1</diffuse>
-          </material>
-        </visual>
-        <inertial>
-          <mass>10</mass>
-          <inertia>
-            <ixx>1</ixx><ixy>0</ixy><ixz>0</ixz>
-            <iyy>1</iyy><iyz>0</iyz>
-            <izz>1</izz>
-          </inertia>
-        </inertial>
-      </link>
-    </model>
     <!-- Laundry area -->
     <include>

File: worlds/rcjo2025_arena.world.xacro (robot description, xacro)
@@ -213,5 +213,5 @@
       <name>bedroom#arm_chair</name>
       <uri>model://arm_chair</uri>
-      <static>false</static>
+      <static>true</static>
       <pose relative_to=''>-2.0 3.25 0.0 0.0 0.0 0.0</pose>
     </include>
