Commit message: [ADD] closed-environment mode for the rcjo frame arenas
Add models/rcjo2025_frame/frame.xacro, a parameterised rcjo2025_frame macro
(wall height, optional ceiling and room lights). precomp2025, rcjo2025 and
rcjo2026 now call it and take a `closed` xacro arg: false keeps the original
open 0.8 m frame, true builds 2.5 m walls with a ceiling and lights.

model.sdf is regenerated at the closed settings so anything still loading
model://rcjo2025_frame keeps working.

File: worlds/precomp2025_arena.world.xacro (robot description, xacro)
@@ -5,4 +5,9 @@
   <xacro:arg name="trofast_knob" default="true" />
   <xacro:arg name="highrtf" default="false" />
+  <!-- closed:=true -> 2.5 m walls + ceiling + lights;
+       false keeps the original open 0.8 m frame. -->
+  <xacro:arg name="closed" default="false" />
+  <xacro:property name="closed" value="$(arg closed)" />
+  <xacro:include filename="$(find sobits_gazebo_worlds)/models/rcjo2025_frame/frame.xacro" />
   <world name='rcjo2025_arena'>
     <plugin
@@ -107,10 +112,7 @@
       <pose relative_to=''>-5 -5 0 0 0 0</pose>
     </include>
-    <include>
-      <name>rcjo2025_frame</name>
-      <static>1</static>
-      <uri>model://rcjo2025_frame</uri>
-      <pose relative_to=''>0 0 0 0 0 0</pose>
-    </include>
+    <xacro:rcjo2025_frame name="rcjo2025_frame"
+                          wall_h="${2.5 if closed else 0.8}"
+                          ceiling="${closed}" lights="${closed}"/>
     <!-- Global Models -->
     <!-- Living Room -->

File: worlds/rcjo2025_arena.world.xacro (robot description, xacro)
@@ -5,4 +5,9 @@
   <xacro:arg name="trofast_knob" default="true" />
   <xacro:arg name="highrtf" default="false" />
+  <!-- closed:=true -> 2.5 m walls + ceiling + lights;
+       false keeps the original open 0.8 m frame. -->
+  <xacro:arg name="closed" default="false" />
+  <xacro:property name="closed" value="$(arg closed)" />
+  <xacro:include filename="$(find sobits_gazebo_worlds)/models/rcjo2025_frame/frame.xacro" />
   <world name='rcjo2025_arena'>
     <plugin
@@ -107,10 +112,7 @@
       <pose relative_to=''>-5 -5 0 0 0 0</pose>
     </include>
-    <include>
-      <name>rcjo2025_frame</name>
-      <static>1</static>
-      <uri>model://rcjo2025_frame</uri>
-      <pose relative_to=''>0 0 0 0 0 0</pose>
-    </include>
+    <xacro:rcjo2025_frame name="rcjo2025_frame"
+                          wall_h="${2.5 if closed else 0.8}"
+                          ceiling="${closed}" lights="${closed}"/>
     <!-- Global Models -->
     <!-- Living Room -->
